Commit message: Fixed issue with ros control and initialization

File: mirte_description/urdf/mirte_arm.urdf (robot description, URDF)
Before this commit: robot mearm, 6 links, 5 joints
Joints:
- joint arm: limit lower=-1.57 upper=0.0 effort=30 velocity=1.0 -> lower=-1.57 upper=1.57 effort=30 velocity=10.0
