Commit message: Added ROS2 control for the Arm

File: mirte_description/mirte_master_description/urdf/ros2_control.xacro (robot description, xacro)
@@ -1,4 +1,88 @@
 <?xml version="1.0"?>
 <robot xmlns:xacro="http://www.ros.org/wiki/xacro">
+<!--
+<ros2_control name="ros2_arm_control" type="system">
+      <hardware>
+        <plugin>mirte_master_arm_control/MirteMasterArmHWInterface</plugin>
+        <param name="example_param_hw_start_duration_sec">0</param>
+        <param name="example_param_hw_stop_duration_sec">3.0</param>
+        <param name="example_param_hw_slowdown">1</param>
+      </hardware>
+   <joint name="arm_Rot_joint">
+        <command_interface name="position"/>
+        <state_interface name="position"/>
+        <state_interface name="velocity" />
+   </joint>
+    <joint name="arm_Shoulder_joint">
+        <command_interface name="position"/>
+        <state_interface name="position">
+          <param name="initial_value">-1.56</param>
+        </state_interface>
+        <state_interface name="velocity" />
+    </joint>
+    <joint name="arm_Elbow_joint">
+        <command_interface name="position"/>
+        <state_interface name="position">
+          <param name="initial_value">-1.56</param>
+        </state_interface>
+        <state_interface name="velocity" />
+    </joint>
+    <joint name="arm_Wrist_joint">
+        <command_interface name="position"/>
+        <state_interface name="position">
+          <param name="initial_value">1.56</param>
+        </state_interface>
+        <state_interface name="velocity" />
+    </joint>
+</ros2_control>
+-->
+<ros2_control name="ros2_gripper_control" type="system">
+     <hardware>
+        <plugin>mirte_master_arm_control/MirteMasterArmHWInterface</plugin>
+        <param name="example_param_hw_start_duration_sec">0</param>
+        <param name="example_param_hw_stop_duration_sec">3.0</param>
+        <param name="example_param_hw_slowdown">2</param>
+      </hardware>
+    <joint name="Gripper_joint">
+        <command_interface name="position"/>
+        <state_interface name="position" />
+        <state_interface name="velocity" />
+    </joint>
+<!-- These are only needed in the simulation! -->
+<!--
+    <joint name="_Gripper_joint_r">
+        <param name="mimic">Gripper_joint</param>
+        <param name="multiplier">-1</param>
+        <command_interface name="position"/>
+        <state_interface name="position" />
+        <state_interface name="velocity" />
+    </joint>
+    <joint name="_gripper_link_joint_l">
+        <param name="mimic">Gripper_joint</param>
+        <param name="multiplier">-1.4</param>
+        <command_interface name="position"/>
+        <state_interface name="position" />
+        <state_interface name="velocity" />
+    </joint>
+    <joint name="_gripper_link_joint_r">
+        <param name="mimic">Gripper_joint</param>
+        <param name="multiplier">1.4</param>
+        <command_interface name="position"/>
+        <state_interface name="position" />
+        <state_interface name="velocity" />
+    </joint>
+    <joint name="gripper_finger_joint_l">
+        <command_interface name="position"/>
+        <state_interface name="position" />
+        <state_interface name="velocity" />
+    </joint>
+    <joint name="gripper_finger_joint_r">
+        <command_interface name="position"/>
+        <state_interface name="position" />
+        <state_interface name="velocity" />
+    </joint>
+-->
+</ros2_control>
+<!--
   <ros2_control name="GazeboSystem" type="system">
     <hardware>
@@ -41,19 +125,26 @@
         <state_interface name="effort" />
     </joint>
+    <xacro:if value="$(arg arm_enable)">
     <joint name="arm_Rot_joint">
         <command_interface name="position"/>
-        <state_interface name="position" />
-    </joint>
+        <state_interface name="position"/>
+   </joint>
     <joint name="arm_Shoulder_joint">
         <command_interface name="position"/>
-        <state_interface name="position" />
+        <state_interface name="position">
+          <param name="initial_value">-1.56</param>
+        </state_interface>
     </joint>
     <joint name="arm_Elbow_joint">
         <command_interface name="position"/>
-        <state_interface name="position" />
+        <state_interface name="position">
+          <param name="initial_value">-1.56</param>
+        </state_interface>
     </joint>
     <joint name="arm_Wrist_joint">
         <command_interface name="position"/>
-        <state_interface name="position" />
+        <state_interface name="position">
+          <param name="initial_value">1.56</param>
+        </state_interface>
     </joint>
     <joint name="Gripper_joint">
@@ -61,8 +152,39 @@
         <state_interface name="position" />
     </joint>
+    <joint name="_Gripper_joint_r">
+        <param name="mimic">Gripper_joint</param>
+        <param name="multiplier">-1</param>
+        <command_interface name="position"/>
+        <state_interface name="position" />
+    </joint>
+    <joint name="_gripper_link_joint_l">
+        <param name="mimic">Gripper_joint</param>
+        <param name="multiplier">-1.4</param>
+        <command_interface name="position"/>
+        <state_interface name="position" />
+    </joint>
+    <joint name="_gripper_link_joint_r">
+        <param name="mimic">Gripper_joint</param>
+        <param name="multiplier">1.4</param>
+        <command_interface name="position"/>
+        <state_interface name="position" />
+    </joint>
+    <joint name="gripper_finger_joint_l">
+        <command_interface name="position"/>
+        <state_interface name="position" />
+    </joint>
+    <joint name="gripper_finger_joint_r">
+        <command_interface name="position"/>
+        <state_interface name="position" />
+    </joint>
+    </xacro:if>
   </ros2_control>
+-->
 <gazebo>
     <plugin filename="libgazebo_ros2_control.so" name="gazebo_ros2_control">
        <parameters>$(find mirte_master_description)/config/mirte_base_control.yaml</parameters>
+       <xacro:if value="$(arg arm_enable)">
+          <parameters>$(find mirte_master_description)/config/mirte_arm_control.yaml</parameters>
+       </xacro:if>
     </plugin>
     <plugin filename="libgazebo_ros_planar_move.so" name="gazebo_planar_move">
