Commit message: Added ultrasonic sensors

File: mirte_description/mirte_master_description/urdf/mirte_master.xacro (robot description, xacro)
@@ -168,20 +168,20 @@
     </joint>
     <link name="link_chassis" />
-    <xacro:ultrasonic_sensor name="left_front">
+    <xacro:ultrasonic_sensor name="front_left">
       <origin
         xyz="0.05297775289576 -0.120282421780502 -0.031"
         rpy="0 0 ${-pi/2+0.296705972839036}" />
     </xacro:ultrasonic_sensor>
-    <xacro:ultrasonic_sensor name="right_front">
+    <xacro:ultrasonic_sensor name="front_right">
       <origin
         xyz="-0.05297775289576 -0.120282421780502 -0.031"
         rpy="0 0 ${-pi/2-0.296705972839036}" />
     </xacro:ultrasonic_sensor>
-    <xacro:ultrasonic_sensor name="left_rear">
+    <xacro:ultrasonic_sensor name="rear_left">
       <origin
         xyz="0.0565606470918482 0.119187021096338 -0.031"
         rpy="0 0 ${-pi/2 + 2.84488668075076}" />
     </xacro:ultrasonic_sensor>
-    <xacro:ultrasonic_sensor name="right_rear">
+    <xacro:ultrasonic_sensor name="rear_right">
       <origin
         xyz="-0.0565606470918482 0.119187021096338 -0.031"

File: mirte_description/mirte_master_description/urdf/ultrasonic.xacro (robot description, xacro)
@@ -9,7 +9,7 @@
       <xacro:insert_block name="origin"/>
       <parent link="link_chassis"/>
-      <child link="base_sonar_${name}"/>
+      <child link="${name}_sonar"/>
     </joint>
-    <link name="base_sonar_${name}">
+    <link name="${name}_sonar">
       <visual>
         <origin rpy="0 0 ${radians(-90)}" />
@@ -19,6 +19,12 @@
         <material name="blue" />
       </visual>
+      <collision>
+        <origin rpy="0 0 ${radians(-90)}" />
+        <geometry>
+          <box size=".045 .025 .02" />
+        </geometry>
+      </collision>
     </link>
-    <gazebo reference="base_sonar_${name}">
+    <gazebo reference="${name}_sonar">
       <sensor type="ray" name="range_sensor_${name}">
         <visualize>${visualize_sensors}</visualize>

Commit message: Fixes to get Gazebo up and running

File: mirte_description/mirte_master_description/urdf/mirte_master.xacro (robot description, xacro)
@@ -10,4 +10,5 @@
   <xacro:arg name="depth_camera_enable" default="True" />
   <xacro:arg name="imu_enable" default="True" />
+  <xacro:arg name="sim" default="False" />
   <xacro:property name="camera_name" value="camera" lazy_eval="False"/>
   <xacro:property name="namespace" value="" scope="global" lazy_eval="False"/>

File: mirte_description/mirte_master_description/urdf/ros2_control.xacro (robot description, xacro)
@@ -1,19 +1,7 @@
 <?xml version="1.0"?>
 <robot xmlns:xacro="http://www.ros.org/wiki/xacro">
-   <xacro:property name="yaml_param_file" value="$(find mirte_base_control)/config/control_master.yaml"/>
-    <xacro:property name="params" value="${xacro.load_yaml(yaml_param_file)}"/>
+<xacro:property name="yaml_param_file" value="$(find mirte_base_control)/config/control_master.yaml"/>
+<xacro:property name="params" value="${xacro.load_yaml(yaml_param_file)}"/>
 <xacro:arg name="prefix" default="" />
-<xacro:macro name="wheel" params="name prefix">
-    <joint name="${prefix}${name}_wheel_joint" type="continuous">
-      <parent link="${prefix}base_link"/>
-      <child link="${prefix}${name}_wheel"/>
-      <origin xyz="0 0 0" rpy="0 0 0"/>
-      <axis xyz="0 1 0"/>
-      <dynamics damping="0.2"/>
-    </joint>
-    <!-- left wheel Link -->
-    <link name="${prefix}${name}_wheel">
-</link>
-</xacro:macro>
 <xacro:macro name="joint" params="name prefix">
       <joint name="${prefix}${name}_wheel_joint">
@@ -25,21 +13,31 @@
    <ros2_control name="mecanumdrive" type="system">
       <hardware>
-        <plugin>mirte_base_control/MirteBaseHWInterface</plugin>
-        <param name="ticks">${params['ticks']}</param>
-        <param name="enable_pid">${params['enable_pid']}</param>
-        <param name="kp">${params['kp']}</param>
-        <param name="ki">${params['ki']}</param>
-        <param name="kd">${params['kd']}</param>
-        <param name="i_clamp">${params['i_clamp']}</param>
-        <param name="antiwindup">${params['antiwindup']}</param>
+        <xacro:if value="$(arg sim)">
+          <plugin>gazebo_ros2_control/GazeboSystem</plugin>
+        </xacro:if>
+        <xacro:unless value="$(arg sim)">
+          <plugin>mirte_base_control/MirteBaseHWInterface</plugin>
+          <param name="ticks">${params['ticks']}</param>
+          <param name="enable_pid">${params['enable_pid']}</param>
+          <param name="kp">${params['kp']}</param>
+          <param name="ki">${params['ki']}</param>
+          <param name="kd">${params['kd']}</param>
+          <param name="i_clamp">${params['i_clamp']}</param>
+          <param name="antiwindup">${params['antiwindup']}</param>
+        </xacro:unless>
       </hardware>
-      <xacro:joint prefix="$(arg prefix)" name="front_left"  />
-        <xacro:joint prefix="$(arg prefix)" name="front_right"  />
-        <xacro:joint prefix="$(arg prefix)" name="rear_right"  />
-        <xacro:joint prefix="$(arg prefix)" name="rear_left"  />
+        <xacro:joint prefix="$(arg prefix)" name="front_left" />
+        <xacro:joint prefix="$(arg prefix)" name="front_right" />
+        <xacro:joint prefix="$(arg prefix)" name="rear_right" />
+        <xacro:joint prefix="$(arg prefix)" name="rear_left" />
     </ros2_control>
 <ros2_control name="ros2_arm_control" type="system">
       <hardware>
-        <plugin>mirte_master_arm_control/MirteMasterArmHWInterface</plugin>
+        <xacro:if value="$(arg sim)">
+          <plugin>gazebo_ros2_control/GazeboSystem</plugin>
+        </xacro:if>
+        <xacro:unless value="$(arg sim)">
+          <plugin>mirte_master_arm_control/MirteMasterArmHWInterface</plugin>
+        </xacro:unless>
       </hardware>
    <joint name="shoulder_pan_joint">
@@ -72,51 +70,45 @@
 <ros2_control name="ros2_gripper_control" type="system">
      <hardware>
-        <plugin>mirte_master_arm_control/MirteMasterArmHWInterface</plugin>
+        <xacro:if value="$(arg sim)">
+          <plugin>gazebo_ros2_control/GazeboSystem</plugin>
+        </xacro:if>
+        <xacro:unless value="$(arg sim)">
+          <plugin>mirte_master_arm_control/MirteMasterArmHWInterface</plugin>
+        </xacro:unless>
       </hardware>
     <joint name="gripper_joint">
-        <command_interface name="position"/>
+        <command_interface name="position" />
         <state_interface name="position" />
         <state_interface name="velocity" />
     </joint>
-<!-- These are only needed in the simulation! -->
-<!--
-    <joint name="_Gripper_joint_r">
-        <param name="mimic">Gripper_joint</param>
+    <xacro:if value="$(arg sim)">
+      <joint name="_Gripper_joint_r">
+        <param name="mimic">gripper_joint</param>
         <param name="multiplier">-1</param>
         <command_interface name="position"/>
         <state_interface name="position" />
         <state_interface name="velocity" />
-    </joint>
-    <joint name="_gripper_link_joint_l">
-        <param name="mimic">Gripper_joint</param>
+      </joint>
+      <joint name="_gripper_link_joint_l">
+        <param name="mimic">gripper_joint</param>
         <param name="multiplier">-1.4</param>
         <command_interface name="position"/>
         <state_interface name="position" />
         <state_interface name="velocity" />
-    </joint>
-    <joint name="_gripper_link_joint_r">
-        <param name="mimic">Gripper_joint</param>
+      </joint>
+      <joint name="_gripper_link_joint_r">
+        <param name="mimic">gripper_joint</param>
         <param name="multiplier">1.4</param>
         <command_interface name="position"/>
         <state_interface name="position" />
         <state_interface name="velocity" />
-    </joint>
-    <joint name="gripper_finger_joint_l">
-        <command_interface name="position"/>
-        <state_interface name="position" />
-        <state_interface name="velocity" />
-    </joint>
-    <joint name="gripper_finger_joint_r">
-        <command_interface name="position"/>
-        <state_interface name="position" />
-        <state_interface name="velocity" />
-    </joint>
--->
+      </joint>
+    </xacro:if>
 </ros2_control>
 <gazebo>
     <plugin filename="libgazebo_ros2_control.so" name="gazebo_ros2_control">
-       <parameters>$(find mirte_master_description)/config/mirte_base_control.yaml</parameters>
+       <parameters>$(find mirte_base_control)/config/mirte_base_control.yaml</parameters>
        <xacro:if value="$(arg arm_enable)">
-          <parameters>$(find mirte_master_description)/config/mirte_arm_control.yaml</parameters>
+          <parameters>$(find mirte_master_arm_control)/config/mirte_master_arm_control.yaml</parameters>
        </xacro:if>
     </plugin>
