Commit message: Fix lidar location for MMv3, thanks @TheOrange-cmd & @martensgun

File: mirte_description/mirte_master_description/urdf/lidar.xacro (robot description, xacro)
@@ -62,5 +62,5 @@
     <link name="laser"></link>
     <joint name="laser_joint" type="fixed">
-      <origin rpy="0 0 ${radians(90)}" />
+      <origin xyz="-0.1 0 0" rpy="0 0 ${radians(90)}" />
       <parent link="lidar_link" />
       <child link="laser" />

Commit message: Better fix lidar location, thanks @JakaHatlakLJ

File: mirte_description/mirte_master_description/urdf/lidar.xacro (robot description, xacro)
@@ -44,5 +44,5 @@
     type="fixed">
     <origin
-      xyz="0 -0.1005 0.0072113248654052"
+      xyz="0 -0.0005 0.0072113248654052"
       rpy="-1.5707963267949 0 -1.5707963267949" />
     <parent
@@ -62,5 +62,5 @@
     <link name="laser"></link>
     <joint name="laser_joint" type="fixed">
-      <origin xyz="-0.1 0 0" rpy="0 0 ${radians(90)}" />
+      <origin xyz="0 0 0" rpy="0 0 ${radians(90)}" />
       <parent link="lidar_link" />
       <child link="laser" />
