Commit message: Modified values to float for moveit, created correct wheel X config, using correct STLs

File: mirte_description/mirte_master_description/urdf/arm.xacro (robot description, xacro)
@@ -23,5 +23,5 @@
             <geometry>
                 <mesh
-                    filename="file://$(find mirte_master_description)/meshes/arm_Rot.STL" />
+                    filename="package://mirte_master_description/meshes/arm_Rot.STL" />
             </geometry>
             <material
@@ -37,5 +37,5 @@
             <geometry>
                 <mesh
-                    filename="file://$(find mirte_master_description)/meshes/arm_Rot.STL" />
+                    filename="package://mirte_master_description/meshes/arm_Rot.STL" />
             </geometry>
         </collision>
@@ -56,6 +56,6 @@
             lower="${pi/-2}"
             upper="${pi/2}"
-            effort="2"
-            velocity="2"
+            effort="2.0"
+            velocity="2.0"
         />
     </joint>
@@ -82,5 +82,5 @@
             <geometry>
                 <mesh
-                    filename="file://$(find mirte_master_description)/meshes/arm_Shoulder.STL" />
+                    filename="package://mirte_master_description/meshes/arm_Shoulder.STL" />
             </geometry>
             <material
@@ -96,5 +96,5 @@
             <geometry>
                 <mesh
-                    filename="file://$(find mirte_master_description)/meshes/arm_Shoulder.STL" />
+                    filename="package://mirte_master_description/meshes/arm_Shoulder.STL" />
             </geometry>
         </collision>
@@ -115,6 +115,6 @@
             lower="${pi/-2}"
             upper="${pi/2}"
-            effort="2"
-            velocity="2"
+            effort="2.0"
+            velocity="2.0"
         />
     </joint>
@@ -141,5 +141,5 @@
             <geometry>
                 <mesh
-                    filename="file://$(find mirte_master_description)/meshes/arm_Elbow.STL" />
+                    filename="package://mirte_master_description/meshes/arm_Elbow.STL" />
             </geometry>
             <material
@@ -155,5 +155,5 @@
             <geometry>
                 <mesh
-                    filename="file://$(find mirte_master_description)/meshes/arm_Elbow.STL" />
+                    filename="package://mirte_master_description/meshes/arm_Elbow.STL" />
             </geometry>
         </collision>
@@ -174,6 +174,6 @@
             lower="${pi/-2}"
             upper="${pi/2}"
-            effort="2"
-            velocity="2"
+            effort="2.0"
+            velocity="2.0"
         />
     </joint>
@@ -200,5 +200,5 @@
             <geometry>
                 <mesh
-                    filename="file://$(find mirte_master_description)/meshes/arm_Wrist.STL" />
+                    filename="package://mirte_master_description/meshes/arm_Wrist.STL" />
             </geometry>
             <material
@@ -214,5 +214,5 @@
             <geometry>
                 <mesh
-                    filename="file://$(find mirte_master_description)/meshes/arm_Wrist.STL" />
+                    filename="package://mirte_master_description/meshes/arm_Wrist.STL" />
             </geometry>
         </collision>
@@ -233,6 +233,6 @@
             lower="${pi/-2}"
             upper="${pi/2}"
-            effort="2"
-            velocity="2"
+            effort="2.0"
+            velocity="2.0"
         />
     </joint>
@@ -259,5 +259,5 @@
             <geometry>
                 <mesh
-                    filename="file://$(find mirte_master_description)/meshes/Gripper.STL" />
+                    filename="package://mirte_master_description/meshes/Gripper.STL" />
             </geometry>
             <material
@@ -273,5 +273,5 @@
             <geometry>
                 <mesh
-                    filename="file://$(find mirte_master_description)/meshes/Gripper.STL" />
+                    filename="package://mirte_master_description/meshes/Gripper.STL" />
             </geometry>
         </collision>
@@ -290,11 +290,11 @@
             xyz="0 -1 0" />
         <limit
-            lower="0"
-            upper="${pi/2}"
-            effort="2"
-            velocity="2"
+            lower="-.20"
+            upper="0.25"
+            effort="2.0"
+            velocity="2.0"
         />
     </joint>
-    <link
+   <link
         name="_gripper_link_r">
         <inertial>
@@ -318,5 +318,5 @@
             <geometry>
                 <mesh
-                    filename="file://$(find mirte_master_description)/meshes/_gripper_link_r.STL" />
+                    filename="package://mirte_master_description/meshes/_gripper_link_r.STL" />
             </geometry>
             <material
@@ -332,5 +332,5 @@
             <geometry>
                 <mesh
-                    filename="file://$(find mirte_master_description)/meshes/_gripper_link_r.STL" />
+                    filename="package://mirte_master_description/meshes/_gripper_link_r.STL" />
             </geometry>
         </collision>
@@ -347,10 +347,11 @@
             link="_gripper_link_r" />
         <axis
-            xyz="0 0 1" />
-        <limit
-            lower="0"
-            upper="0"
-            effort="0"
-            velocity="0" />
+            xyz="0 -1 0" />
+        <limit
+            lower="-3.14"
+            upper="3.14"
+            effort="0.0"
+            velocity="0.0" />
+        <mimic joint="Gripper_joint" multiplier="1.4"/>
     </joint>
     <link
@@ -376,5 +377,5 @@
             <geometry>
                 <mesh
-                    filename="file://$(find mirte_master_description)/meshes/gripper_finger_r.STL" />
+                    filename="package://mirte_master_description/meshes/gripper_finger_r.STL" />
             </geometry>
             <material
@@ -390,5 +391,5 @@
             <geometry>
                 <mesh
-                    filename="file://$(find mirte_master_description)/meshes/gripper_finger_r.STL" />
+                    filename="package://mirte_master_description/meshes/gripper_finger_r.STL" />
             </geometry>
         </collision>
@@ -407,8 +408,8 @@
             xyz="0 0 1" />
         <limit
-            lower="0"
-            upper="0"
-            effort="0"
-            velocity="0" />
+            lower="0.0"
+            upper="0.0"
+            effort="0.0"
+            velocity="0.0" />
     </joint>
     <link
@@ -434,5 +435,5 @@
             <geometry>
                 <mesh
-                    filename="file://$(find mirte_master_description)/meshes/_gripper_link_l.STL" />
+                    filename="package://mirte_master_description/meshes/_gripper_link_l.STL" />
             </geometry>
             <material
@@ -448,5 +449,5 @@
             <geometry>
                 <mesh
-                    filename="file://$(find mirte_master_description)/meshes/_gripper_link_l.STL" />
+                    filename="package://mirte_master_description/meshes/_gripper_link_l.STL" />
             </geometry>
         </collision>
@@ -463,10 +464,11 @@
             link="_gripper_link_l" />
         <axis
-            xyz="0 0 1" />
-        <limit
-            lower="0"
-            upper="0"
-            effort="0"
-            velocity="0" />
+            xyz="0 -1 0" />
+        <limit
+            lower="-3.14"
+            upper="3.14"
+            effort="0.0"
+            velocity="0.0" />
+        <mimic joint="Gripper_joint" multiplier="-1.4"/>
     </joint>
     <link
@@ -492,5 +494,5 @@
             <geometry>
                 <mesh
-                    filename="file://$(find mirte_master_description)/meshes/gripper_finger_l.STL" />
+                    filename="package://mirte_master_description/meshes/gripper_finger_l.STL" />
             </geometry>
             <material
@@ -506,5 +508,5 @@
             <geometry>
                 <mesh
-                    filename="file://$(find mirte_master_description)/meshes/gripper_finger_l.STL" />
+                    filename="package://mirte_master_description/meshes/gripper_finger_l.STL" />
             </geometry>
         </collision>
@@ -523,8 +525,8 @@
             xyz="0 0 1" />
         <limit
-            lower="0"
-            upper="0"
-            effort="0"
-            velocity="0" />
+            lower="0.0"
+            upper="0.0"
+            effort="0.0"
+            velocity="0.0" />
     </joint>
     <link
@@ -550,5 +552,5 @@
             <geometry>
                 <mesh
-                    filename="file://$(find mirte_master_description)/meshes/_Gripper_r.STL" />
+                    filename="package://mirte_master_description/meshes/_Gripper_r.STL" />
             </geometry>
             <material
@@ -564,5 +566,5 @@
             <geometry>
                 <mesh
-                    filename="file://$(find mirte_master_description)/meshes/_Gripper_r.STL" />
+                    filename="package://mirte_master_description/meshes/_Gripper_r.STL" />
             </geometry>
         </collision>
@@ -579,10 +581,32 @@
             link="_Gripper_r" />
         <axis
-            xyz="0 0 1" />
-        <limit
-            lower="0"
-            upper="0"
-            effort="0"
-            velocity="0" />
-    </joint>
+            xyz="0 -1 0" />
+        <limit
+            lower="-.25"
+            upper="0.20"
+            effort="2.0"
+            velocity="2.0"
+        />
+        <mimic joint="Gripper_joint" multiplier="-1"/>
+    </joint>
+<gazebo>
+    <plugin filename="libgazebo_grasp_fix.so" name="gazebo_grasp_fix">
+       <arm>
+          <arm_name>finger_gripper</arm_name>
+          <palm_link>arm_Wrist</palm_link>
+          <gripper_link>Gripper</gripper_link>
+          <gripper_link>_Gripper_r</gripper_link>
+          <gripper_link>_gripper_link_l</gripper_link>
+          <gripper_link>gripper_finger_l</gripper_link>
+          <gripper_link>_gripper_link_r</gripper_link>
+          <gripper_link>gripper_finger_r</gripper_link>
+       </arm>
+       <forces_angle_tolerance>100</forces_angle_tolerance>
+       <update_rate>4</update_rate>
+       <grip_count_threshold>4</grip_count_threshold>
+       <max_grip_count>8</max_grip_count>
+       <release_tolerance>0.005</release_tolerance>
+       <disable_collisions_on_attach>false</disable_collisions_on_attach>
+    </plugin>
+</gazebo>
 </robot>

File: mirte_description/mirte_master_description/urdf/lidar.xacro (robot description, xacro)
@@ -22,5 +22,5 @@
       <geometry>
         <mesh
-          filename="file://$(find mirte_master_description)/meshes/lidar.STL" />
+          filename="package://mirte_master_description/meshes/lidar.STL" />
       </geometry>
       <material
@@ -36,5 +36,5 @@
       <geometry>
         <mesh
-          filename="file://$(find mirte_master_description)/meshes/lidar.STL" />
+          filename="package://mirte_master_description/meshes/lidar.STL" />
       </geometry>
     </collision>
@@ -72,49 +72,8 @@
     <xacro:property name="lidar_sensor_link" value="lidar_link" />
   </xacro:unless>
-<!--
-  <gazebo reference="lidar_link">
-    <sensor type="ray" name="lidar">
-      <xacro:if value="$(arg use_correct_laser_frame)">
-        <pose>0 0 0 0 0 0</pose>
-      </xacro:if>
-      <xacro:unless value="$(arg use_correct_laser_frame)">
-        <pose>0 0 0 0 0 0</pose>
-      </xacro:unless>
-      <visualize>false</visualize>
-      <update_rate>10</update_rate>
-      <ray>
-        <scan>
-          <horizontal>
-            <samples>500</samples>
-            <resolution>1</resolution>
-            <min_angle>${-pi}</min_angle>
-            <max_angle>${pi}</max_angle>
-          </horizontal>
-        </scan>
-        <range>
-          <min>0.05</min>
-          <max>10.0</max>
-          <resolution>0.015</resolution>
-        </range>
-        <noise>
-          <type>gaussian</type>
-          <mean>0.0</mean>
-          <stddev>0.01</stddev>
-        </noise>
-      </ray>
-      <plugin name="gazebo_lidar" filename="libgazebo_ros_laser.so">
-        <ros>
-          <remapping>~/out:=scan</remapping>
-        </ros>
-        <output_type>sensor_msgs/LaserScan</output_type>
-        <frame_name>${lidar_sensor_link}</frame_name>
-      </plugin>
-    </sensor>
-  </gazebo>
--->
   <gazebo reference="lidar_link">
         <sensor name="lidar" type="ray">
             <pose> 0 0 0 0 0 0 </pose>
-            <visualize>false</visualize>
+            <visualize>${visualize_sensors}</visualize>
             <update_rate>10</update_rate>
             <ray>
@@ -128,5 +87,5 @@
                 </scan>
                 <range>
-                    <min>0.02</min>
+                    <min>0.03</min>
                     <max>12</max>
                     <resolution>0.01</resolution>
