Commit message: Modified values to float for moveit, created correct wheel X config, using correct STLs

File: mirte_description/mirte_master_description/urdf/mirte_master.xacro (robot description, xacro)
@@ -6,20 +6,11 @@
   <xacro:arg name="screen_enable" default="False" />
   <xacro:arg name="front_camera_enable" default="False" />
-  <xacro:arg name="sonar_enable" default="False" />
-  <xacro:arg name="lidar_enable" default="False" />
-  <xacro:arg name="depth_camera_enable" default="False" />
-  <xacro:arg name="imu_enable" default="False" />
-  <xacro:arg name="use_namespace" default="False"/>
-  <xacro:arg name="namespace_name" default="" />
-  <xacro:if value="$(arg use_namespace)" >
-    <xacro:property name="camera_name" value="$(arg namespace_name)/camera" lazy_eval="False"/>
-    <xacro:property name="namespace" value="$(arg namespace_name)" scope="global" lazy_eval="False"/>
-    <xacro:property name="tf_namespace" value="$(arg namespace_name)/" scope="global" lazy_eval="False"/>
-  </xacro:if>
-  <xacro:unless value="$(arg use_namespace)">
-    <xacro:property name="camera_name" value="camera" lazy_eval="False"/>
-    <xacro:property name="namespace" value="" scope="global" lazy_eval="False"/>
-    <xacro:property name="tf_namespace" value="" scope="global" lazy_eval="False"/>
-  </xacro:unless>
+  <xacro:arg name="sonar_enable" default="True" />
+  <xacro:arg name="lidar_enable" default="True" />
+  <xacro:arg name="depth_camera_enable" default="True" />
+  <xacro:arg name="imu_enable" default="True" />
+  <xacro:property name="camera_name" value="camera" lazy_eval="False"/>
+  <xacro:property name="namespace" value="" scope="global" lazy_eval="False"/>
+  <xacro:property name="tf_namespace" value="" scope="global" lazy_eval="False"/>
   <xacro:arg name="use_correct_laser_frame" default="True" />
   <xacro:property name="wheel_radius" value="0.050" />
@@ -29,4 +20,5 @@
   <xacro:property name="wheel_effort" value="5" />
   <xacro:property name="base_mass" value="5.0" />
+  <xacro:property name="visualize_sensors" value="True" />
   <material name="blue">
     <color rgba="0.203125 0.23828125 0.28515625 1.0" />
@@ -34,5 +26,6 @@
   <xacro:include filename="$(find mirte_master_description)/urdf/mirte_master_base.gazebo.xacro" />
   <xacro:if value="$(arg depth_camera_enable)">
-    <xacro:sensor_orbbec_astra_pro_plus name="${camera_name}" parent="frame_link" color="black">
+    <xacro:include filename="$(find mirte_master_description)/urdf/orbbec_astra_plus_pro.xacro" />
+    <xacro:sensor_orbbec_astra_pro_plus name="${camera_name}" parent="frame_link" color="blue">
       <origin xyz="0.01 -0.146658788505756 0.0427" rpy="0 0 ${radians(-90)}" />
     </xacro:sensor_orbbec_astra_pro_plus>
@@ -47,4 +40,7 @@
   </xacro:if>
   <link name="base_link" />
+  <gazebo reference="base_link">
+     <kinematic>1</kinematic>
+  </gazebo>
   <joint name="frame_base_joint" type="fixed">
     <origin xyz="0 0 0.10" rpy="0 0 ${radians(90)}" />
@@ -66,5 +62,5 @@
       <geometry>
         <mesh
-          filename="file://$(find mirte_master_description)/meshes/frame_link.STL" />
+          filename="package://mirte_master_description/meshes/frame_link.STL" />
       </geometry>
       <material name="">
@@ -72,40 +68,4 @@
       </material>
     </visual>
-    <visual>
-      <origin
-        xyz="0.05297775289576 -0.120282421780502 -0.031"
-        rpy="3.14159265358979 0 0.296705972839036" />
-      <geometry>
-        <mesh filename="file://$(find mirte_master_description)/meshes/ultrasonic_fl.STL" />
-      </geometry>
-      <material name="blue" />
-    </visual>
-    <visual>
-      <origin
-        xyz="-0.05297775289576 -0.120282421780502 -0.031"
-        rpy="3.14159265358979 0 -0.296705972839036" />
-      <geometry>
-        <mesh filename="file://$(find mirte_master_description)/meshes/ultrasonic_fr.STL" />
-      </geometry>
-      <material name="blue" />
-    </visual>
-    <visual>
-      <origin
-        xyz="0.0565606470918482 0.119187021096338 -0.031"
-        rpy="3.14159265358979 0 2.84488668075076" />
-      <geometry>
-        <mesh filename="file://$(find mirte_master_description)/meshes/ultrasonic_bl.STL" />
-      </geometry>
-      <material name="blue" />
-    </visual>
-    <visual>
-      <origin
-        xyz="-0.0565606470918482 0.119187021096338 -0.031"
-        rpy="3.14159265358979 0 -2.84488668075076" />
-      <geometry>
-        <mesh filename="file://$(find mirte_master_description)/meshes/ultrasonic_br.STL" />
-      </geometry>
-      <material name="blue" />
-    </visual>
     <collision>
       <origin xyz="0 0 -0.03" />
@@ -133,188 +93,29 @@
     </collision>
   </link>
-  <link
-    name="wheel_left_front">
-    <inertial>
-      <origin xyz="0 0 0.025" />
-      <mass value="${wheel_mass}" />
-      <inertia
-        ixx="${wheel_mass * (3 * (wheel_radius**2) + (wheel_length**2)) / 12}"
-        iyy="${wheel_mass * (3 * (wheel_radius**2) + (wheel_length**2)) / 12}"
-        izz="${wheel_mass * (wheel_radius **2) / 2}"
-        ixy="0" ixz="0" iyz="0" />
-    </inertial>
-    <visual>
-      <geometry>
-        <mesh
-          filename="file://$(find mirte_master_description)/meshes/wheel_left_front.STL" />
-      </geometry>
-      <material name="">
-        <color rgba="0.79216 0.81961 0.93333 1" />
-      </material>
-    </visual>
-    <collision>
-      <origin xyz="0 0 0.025" />
-      <geometry>
-        <cylinder radius="${wheel_radius}" length="${wheel_length}" />
-      </geometry>
-    </collision>
-  </link>
-  <joint
-    name="wheel_left_front_joint"
-    type="continuous">
-    <origin
-      xyz="0.153 -0.085 -0.0455"
-      rpy="1.5708 0 -1.5708" />
-    <parent link="frame_link" />
-    <child link="wheel_left_front" />
-    <axis xyz="0 0 -1" />
-  </joint>
-  <transmission name="wheel_left_front_transmission">
-    <type>transmission_interface/SimpleTransmission</type>
-    <joint name="wheel_left_front_joint">
-      <hardwareInterface>hardware_interface/VelocityJointInterface</hardwareInterface>
-    </joint>
-    <actuator name="wheel_left_front_actuator">
-      <mechanicalReduction>1</mechanicalReduction>
-    </actuator>
-  </transmission>
-  <link
-    name="wheel_left_rear">
-    <inertial>
-      <origin xyz="0 0 0.025" />
-      <mass value="${wheel_mass}" />
-      <inertia
-        ixx="${wheel_mass * (3 * (wheel_radius**2) + (wheel_length**2)) / 12}"
-        iyy="${wheel_mass * (3 * (wheel_radius**2) + (wheel_length**2)) / 12}"
-        izz="${wheel_mass * (wheel_radius **2) / 2}"
-        ixy="0" ixz="0" iyz="0" />
-    </inertial>
-    <visual>
-      <geometry>
-        <mesh
-          filename="file://$(find mirte_master_description)/meshes/wheel_left_rear.STL" />
-      </geometry>
-      <material name="">
-        <color rgba="0.79216 0.81961 0.93333 1" />
-      </material>
-    </visual>
-    <collision>
-      <origin xyz="0 0 0.025" />
-      <geometry>
-        <cylinder radius="${wheel_radius}" length="${wheel_length}" />
-      </geometry>
-    </collision>
-  </link>
-  <joint
-    name="wheel_left_rear_joint"
-    type="continuous">
-    <origin
-      xyz="0.153 0.085 -0.0455"
-      rpy="1.5708 0 -1.5708" />
-    <parent link="frame_link" />
-    <child link="wheel_left_rear" />
-    <axis xyz="0 0 -1" />
-  </joint>
-  <transmission name="wheel_left_rear_transmission">
-    <type>transmission_interface/SimpleTransmission</type>
-    <joint name="wheel_left_rear_joint">
-      <hardwareInterface>hardware_interface/VelocityJointInterface</hardwareInterface>
-    </joint>
-    <actuator name="wheel_left_rear_actuator">
-      <mechanicalReduction>1</mechanicalReduction>
-    </actuator>
-  </transmission>
-  <link
-    name="wheel_right_front">
-    <inertial>
-      <origin xyz="0 0 -0.025" />
-      <mass value="${wheel_mass}" />
-      <inertia
-        ixx="${wheel_mass * (3 * (wheel_radius**2) + (wheel_length**2)) / 12}"
-        iyy="${wheel_mass * (3 * (wheel_radius**2) + (wheel_length**2)) / 12}"
-        izz="${wheel_mass * (wheel_radius **2) / 2}"
-        ixy="0" ixz="0" iyz="0" />
-    </inertial>
-    <visual>
-      <geometry>
-        <mesh
-          filename="file://$(find mirte_master_description)/meshes/wheel_right_front.STL" />
-      </geometry>
-      <material name="">
-        <color rgba="0.79216 0.81961 0.93333 1" />
-      </material>
-    </visual>
-    <collision>
-      <origin xyz="0 0 -0.025" />
-      <geometry>
-        <cylinder radius="${wheel_radius}" length="${wheel_length}" />
-      </geometry>
-    </collision>
-  </link>
-  <joint
-    name="wheel_right_front_joint"
-    type="continuous">
-    <origin
-      xyz="-0.153 -0.085 -0.0455"
-      rpy="1.5708 0 -1.5708" />
-    <parent link="frame_link" />
-    <child link="wheel_right_front" />
-    <axis xyz="0 0 -1" />
-  </joint>
-  <transmission name="wheel_right_front_transmission">
-    <type>transmission_interface/SimpleTransmission</type>
-    <joint name="wheel_right_front_joint">
-      <hardwareInterface>hardware_interface/VelocityJointInterface</hardwareInterface>
-    </joint>
-    <actuator name="wheel_right_front_actuator">
-      <mechanicalReduction>1</mechanicalReduction>
-    </actuator>
-  </transmission>
-  <link
-    name="wheel_right_rear">
-    <inertial>
-      <origin xyz="0 0 -0.025" />
-      <mass value="${wheel_mass}" />
-      <inertia
-        ixx="${wheel_mass * (3 * (wheel_radius**2) + (wheel_length**2)) / 12}"
-        iyy="${wheel_mass * (3 * (wheel_radius**2) + (wheel_length**2)) / 12}"
-        izz="${wheel_mass * (wheel_radius **2) / 2}"
-        ixy="0" ixz="0" iyz="0" />
-    </inertial>
-    <visual>
-      <geometry>
-        <mesh
-          filename="file://$(find mirte_master_description)/meshes/wheel_right_rear.STL" />
-      </geometry>
-      <material name="">
-        <color rgba="0.79216 0.81961 0.93333 1" />
-      </material>
-    </visual>
-    <collision>
-      <origin xyz="0 0 -0.025" />
-      <geometry>
-        <cylinder radius="${wheel_radius}" length="${wheel_length}" />
-      </geometry>
-    </collision>
-  </link>
-  <joint
-    name="wheel_right_rear_joint"
-    type="continuous">
-    <origin
-      xyz="-0.153 0.085 -0.0455"
-      rpy="1.5708 0 -1.5708" />
-    <parent link="frame_link" />
-    <child link="wheel_right_rear" />
-    <axis xyz="0 0 -1" />
-  </joint>
-  <transmission name="wheel_right_rear_transmission">
-    <type>transmission_interface/SimpleTransmission</type>
-    <joint name="wheel_right_rear_joint">
-      <hardwareInterface>hardware_interface/VelocityJointInterface</hardwareInterface>
-    </joint>
-    <actuator name="wheel_right_rear_actuator">
-      <mechanicalReduction>1</mechanicalReduction>
-    </actuator>
-  </transmission>
+  <xacro:include filename="$(find mirte_master_description)/urdf/wheel.xacro" />
+   <!-- 0.025   -1 -->
+    <xacro:mecanum_wheel name="left_front" wheel_type="left" link_origin="0.025">
+      <origin
+        xyz="${0.153 - 0} -0.085 -0.0455"
+        rpy="1.5708 0 -1.5708" />
+    </xacro:mecanum_wheel>
+   <!-- 0.025   -1 -->
+    <xacro:mecanum_wheel name="left_rear" wheel_type="right" link_origin="0.025">
+      <origin
+        xyz="${0.153 - 0} 0.085 -0.0455"
+        rpy="1.5708 0 -1.5708" />
+    </xacro:mecanum_wheel>
+   <!-- -0.025   -1 -->
+    <xacro:mecanum_wheel name="right_front" wheel_type="right" link_origin="-0.025">
+      <origin
+        xyz="${-0.153 + wheel_length} -0.085 -0.0455"
+        rpy="1.5708 0 -1.5708" />
+    </xacro:mecanum_wheel>
+   <!-- -0.025   -1 -->
+    <xacro:mecanum_wheel name="right_rear" wheel_type="left" link_origin="-0.025">
+      <origin
+        xyz="${-0.153 + wheel_length} 0.085 -0.0455"
+        rpy="1.5708 0 -1.5708" />
+    </xacro:mecanum_wheel>
   <xacro:if value="$(arg front_camera_enable)">
     <link
@@ -340,5 +141,5 @@
         <geometry>
           <mesh
-            filename="file://$(find mirte_master_description)/meshes/cam_front.STL" />
+            filename="package://mirte_master_description/meshes/cam_front.STL" />
         </geometry>
         <material
@@ -414,5 +215,5 @@
         <geometry>
           <mesh
-            filename="file://$(find mirte_master_description)/meshes/screen.STL" />
+            filename="package://mirte_master_description/meshes/screen.STL" />
         </geometry>
         <material
@@ -428,5 +229,5 @@
         <geometry>
           <mesh
-            filename="file://$(find mirte_master_description)/meshes/screen.STL" />
+            filename="package://mirte_master_description/meshes/screen.STL" />
         </geometry>
       </collision>

File: mirte_description/mirte_master_description/urdf/ultrasonic.xacro (robot description, xacro)
@@ -12,63 +12,55 @@
     </joint>
     <link name="base_sonar_${name}">
-      <!-- <collision>
-        <origin xyz="0 0 0" rpy="0 0 0"/>
+      <visual>
+        <origin rpy="0 0 ${radians(-90)}" />
         <geometry>
-          <box size="0.01 0.05 0.037"/>
+          <mesh filename="package://mirte_master_description/meshes/ultrasonic_fl.STL" />
         </geometry>
-      </collision> -->
-      <visual>
-        <origin xyz="0 0 0" rpy="0 0 0"/>
-        <geometry>
-          <box size="0.01 0.05 0.037"/>
-        </geometry>
-        <material name="blue"/>
+        <material name="blue" />
       </visual>
-      <!-- <inertial>
-        <mass value="0.0"/>
-        <origin xyz="0 0 0" rpy="0 0 0"/>
-        <inertia ixx="0.0" ixy="0.0" ixz="0.0" iyy="0.0" iyz="0.0" izz="0.0"/>
-      </inertial> -->
     </link>
-<!--
     <gazebo reference="base_sonar_${name}">
       <sensor type="ray" name="range_sensor_${name}">
-        <visualize>false</visualize>
-        <ray>
-          <scan>
-            <horizontal>
-              <samples>4</samples>
+        <visualize>${visualize_sensors}</visualize>
+          <ray>
+            <scan>
+              <horizontal>
+                <!-- for some reason 1 does not work, we neex 2x2 -->
+                <samples>2</samples>
+                <resolution>1</resolution>
+                <min_angle>-0.26</min_angle>
+                <max_angle>0.26</max_angle>
+              </horizontal>
+            <vertical>
+              <samples>2</samples>
               <resolution>1</resolution>
-              <min_angle>${-sonar_angle_max/2}</min_angle>
-              <max_angle>${sonar_angle_max/2}</max_angle>
-            </horizontal>
-            <vertical>
-              <samples>4</samples>
-              <resolution>1</resolution>
-              <min_angle>0</min_angle>
-              <max_angle>${sonar_angle_max/4}</max_angle>
+              <min_angle>-0.014835</min_angle>
+              <max_angle>0.014835</max_angle>
             </vertical>
-          </scan>
-          <range>
-            <min>0.025</min>
-            <max>5</max>
-            <resolution>0.01</resolution>
-          </range>
-          <noise>
-            <type>gaussian</type>
-            <mean>0.0</mean>
-            <stddev>0.01</stddev>
-          </noise>
-        </ray>
-        <update_rate>30</update_rate>
-        <plugin name="laser_controller_sonar${name}" filename="libgazebo_ros_laser.so">
-          <topicName>mirte/scanSonar${name}</topicName>
-          <output_type>sensor_msgs/Range</output_type>
-          <radiation_type>ultrasound</radiation_type>
-          <frameName>base_sonar_${name}</frameName>
-        </plugin>
-      </sensor>
-    </gazebo>
- -->
+         </scan>
+         <range>
+           <min>0.03</min>
+           <max>4</max>
+           <resolution>0.01</resolution>
+         </range>
+         <!-- Using gazebo's noise instead of plugin's -->
+         <noise>
+           <type>gaussian</type>
+           <mean>0.0</mean>
+           <stddev>0.01</stddev>
+         </noise>
+       </ray>
+       <!-- Using gazebo's update rate instead of plugin's -->
+       <update_rate>30</update_rate>
+       <plugin name="gazebo_ros_range_controller_${name}" filename="libgazebo_ros_ray_sensor.so">
+         <ros>
+           <namespace>/mirte</namespace>
+           <remapping>~/out:=distance/${name}</remapping>
+         </ros>
+         <output_type>sensor_msgs/Range</output_type>
+         <radiation_type>ultrasound</radiation_type>
+       </plugin>
+     </sensor>
+   </gazebo>
   </xacro:macro>
 </robot>

Commit message: Modified names of arm joints

File: mirte_description/mirte_master_description/urdf/arm.xacro (robot description, xacro)
@@ -2,5 +2,5 @@
 <robot xmlns:xacro="http://www.ros.org/wiki/xacro">
     <link
-        name="arm_Rot">
+        name="arm_shoulder_pan">
         <inertial>
             <origin
@@ -42,5 +42,5 @@
     </link>
     <joint
-        name="arm_Rot_joint"
+        name="arm_shoulder_pan_joint"
         type="revolute">
         <origin
@@ -50,5 +50,5 @@
             link="frame_link" />
         <child
-            link="arm_Rot" />
+            link="arm_shoulder_pan" />
         <axis
             xyz="0 1 0" />
@@ -61,5 +61,5 @@
     </joint>
     <link
-        name="arm_Shoulder">
+        name="arm_shoulder_lift">
         <inertial>
             <origin
@@ -101,5 +101,5 @@
     </link>
     <joint
-        name="arm_Shoulder_joint"
+        name="arm_shoulder_lift_joint"
         type="revolute">
         <origin
@@ -107,7 +107,7 @@
             rpy="3.1416 0 1.5708" />
         <parent
-            link="arm_Rot" />
-        <child
-            link="arm_Shoulder" />
+            link="arm_shoulder_pan" />
+        <child
+            link="arm_shoulder_lift" />
         <axis
             xyz="0 1 0" />
@@ -120,5 +120,5 @@
     </joint>
     <link
-        name="arm_Elbow">
+        name="arm_elbow">
         <inertial>
             <origin
@@ -160,5 +160,5 @@
     </link>
     <joint
-        name="arm_Elbow_joint"
+        name="arm_elbow_joint"
         type="revolute">
         <origin
@@ -166,7 +166,7 @@
             rpy="-3.1416 0 1.5708" />
         <parent
-            link="arm_Shoulder" />
-        <child
-            link="arm_Elbow" />
+            link="arm_shoulder_lift" />
+        <child
+            link="arm_elbow" />
         <axis
             xyz="1 0 0" />
@@ -179,5 +179,5 @@
     </joint>
     <link
-        name="arm_Wrist">
+        name="arm_wrist">
         <inertial>
             <origin
@@ -219,5 +219,5 @@
     </link>
     <joint
-        name="arm_Wrist_joint"
+        name="arm_wrist_joint"
         type="revolute">
         <origin
@@ -225,7 +225,7 @@
             rpy="3.1416 0 1.5708" />
         <parent
-            link="arm_Elbow" />
-        <child
-            link="arm_Wrist" />
+            link="arm_elbow" />
+        <child
+            link="arm_wrist" />
         <axis
             xyz="0 1 0" />
@@ -238,5 +238,5 @@
     </joint>
     <link
-        name="Gripper">
+        name="gripper">
         <inertial>
             <origin
@@ -278,5 +278,5 @@
     </link>
     <joint
-        name="Gripper_joint"
+        name="gripper_joint"
         type="revolute">
         <origin
@@ -284,7 +284,7 @@
             rpy="-1.5708 0 0" />
         <parent
-            link="arm_Wrist" />
-        <child
-            link="Gripper" />
+            link="arm_wrist" />
+        <child
+            link="gripper" />
         <axis
             xyz="0 -1 0" />
@@ -343,5 +343,5 @@
             rpy="1.5708 0 -1.3641" />
         <parent
-            link="arm_Wrist" />
+            link="arm_wrist" />
         <child
             link="_gripper_link_r" />
@@ -460,5 +460,5 @@
             rpy="1.5708 0 -1.7775" />
         <parent
-            link="arm_Wrist" />
+            link="arm_wrist" />
         <child
             link="_gripper_link_l" />
@@ -577,5 +577,5 @@
             rpy="-1.5708 0 -3.1416" />
         <parent
-            link="arm_Wrist" />
+            link="arm_wrist" />
         <child
             link="_Gripper_r" />
@@ -588,5 +588,5 @@
             velocity="2.0"
         />
-        <mimic joint="Gripper_joint" multiplier="-1"/>
+        <mimic joint="gripper_joint" multiplier="-1"/>
     </joint>
 <gazebo>
@@ -594,6 +594,6 @@
        <arm>
           <arm_name>finger_gripper</arm_name>
-          <palm_link>arm_Wrist</palm_link>
-          <gripper_link>Gripper</gripper_link>
+          <palm_link>arm_wrist</palm_link>
+          <gripper_link>gripper</gripper_link>
           <gripper_link>_Gripper_r</gripper_link>
           <gripper_link>_gripper_link_l</gripper_link>

File: mirte_description/mirte_master_description/urdf/ros2_control.xacro (robot description, xacro)
@@ -9,24 +9,24 @@
         <param name="example_param_hw_slowdown">1</param>
       </hardware>
-   <joint name="arm_Rot_joint">
+   <joint name="arm_shoulder_pan_joint">
         <command_interface name="position"/>
         <state_interface name="position"/>
         <state_interface name="velocity" />
    </joint>
-    <joint name="arm_Shoulder_joint">
-        <command_interface name="position"/>
-        <state_interface name="position">
-          <param name="initial_value">-1.56</param>
-        </state_interface>
-        <state_interface name="velocity" />
-    </joint>
-    <joint name="arm_Elbow_joint">
-        <command_interface name="position"/>
-        <state_interface name="position">
-          <param name="initial_value">-1.56</param>
-        </state_interface>
-        <state_interface name="velocity" />
-    </joint>
-    <joint name="arm_Wrist_joint">
+    <joint name="arm_shoulder_lift_joint">
+        <command_interface name="position"/>
+        <state_interface name="position">
+          <param name="initial_value">-1.56</param>
+        </state_interface>
+        <state_interface name="velocity" />
+    </joint>
+    <joint name="arm_elbow_joint">
+        <command_interface name="position"/>
+        <state_interface name="position">
+          <param name="initial_value">-1.56</param>
+        </state_interface>
+        <state_interface name="velocity" />
+    </joint>
+    <joint name="arm_wrist_joint">
         <command_interface name="position"/>
         <state_interface name="position">
@@ -44,5 +44,5 @@
         <param name="example_param_hw_slowdown">2</param>
       </hardware>
-    <joint name="Gripper_joint">
+    <joint name="gripper_joint">
         <command_interface name="position"/>
         <state_interface name="position" />
