Commit message: Fix for fingers not attaching when state broadcasted through ros2 control

File: mirte_description/mirte_master_description/urdf/arm.xacro (robot description, xacro)
@@ -397,5 +397,5 @@
     <joint
         name="gripper_finger_joint_r"
-        type="revolute">
+        type="fixed">
         <origin
             xyz="0 0.01 -0.037"
@@ -407,9 +407,4 @@
         <axis
             xyz="0 0 1" />
-        <limit
-            lower="0.0"
-            upper="0.0"
-            effort="0.0"
-            velocity="0.0" />
     </joint>
     <link
@@ -514,5 +509,5 @@
     <joint
         name="gripper_finger_joint_l"
-        type="revolute">
+        type="fixed">
         <origin
             xyz="0 0 -0.037"
@@ -524,9 +519,4 @@
         <axis
             xyz="0 0 1" />
-        <limit
-            lower="0.0"
-            upper="0.0"
-            effort="0.0"
-            velocity="0.0" />
     </joint>
     <link

Commit message: mimic joints if using sim, but moveit needs arg

File: mirte_description/mirte_master_description/urdf/arm.xacro (robot description, xacro)
@@ -1,4 +1,21 @@
 <?xml version="1.0" encoding="UTF-8"?>
 <robot xmlns:xacro="http://www.ros.org/wiki/xacro">
+<xacro:if value="$(arg sim)">
+<joint name="_gripper_link_joint_r_mimic" type="fixed">
+  <parent link="shoulder_pan" />
+  <child link="random1" />
+</joint>
+<link name="random1"/>
+<joint name="_gripper_link_joint_l_mimic" type="fixed">
+  <parent link="shoulder_pan" />
+  <child link="random2" />
+</joint>
+<link name="random2"/>
+<joint name="_Gripper_joint_r_mimic" type="fixed">
+  <parent link="shoulder_pan" />
+  <child link="random" />
+</joint>
+<link name="random"/>
+</xacro:if>
     <link
         name="shoulder_pan">

Commit message: gz support
Signed-off-by: Juancams <jc.manzanares.serrano@gmail.com>

File: mirte_description/mirte_master_description/urdf/arm.xacro (robot description, xacro)
@@ -353,5 +353,4 @@
             effort="0.0"
             velocity="0.0" />
-        <mimic joint="gripper_joint" multiplier="1.4"/>
     </joint>
     <link
@@ -465,5 +464,4 @@
             effort="0.0"
             velocity="0.0" />
-        <mimic joint="gripper_joint" multiplier="-1.4"/>
     </joint>
     <link
@@ -578,5 +576,4 @@
             velocity="2.0"
         />
-        <mimic joint="gripper_joint" multiplier="-1"/>
     </joint>
 <gazebo>

File: mirte_description/mirte_master_description/urdf/lidar.xacro (robot description, xacro)
@@ -72,10 +72,16 @@
     <xacro:property name="lidar_sensor_link" value="lidar_link" />
   </xacro:unless>
+  <plugin
+    filename="gz-sim-sensors-system"
+    name="gz::sim::systems::Sensors">
+    <render_engine>ogre2</render_engine>
+  </plugin>
   <gazebo reference="lidar_link">
-        <sensor name="lidar" type="ray">
-            <pose> 0 0 0 0 0 0 </pose>
+        <sensor name="lidar" type="gpu_lidar">
+            <always_on>true</always_on>
             <visualize>${visualize_sensors}</visualize>
             <update_rate>10</update_rate>
-            <ray>
+            <topic>scan</topic>
+            <lidar>
                 <scan>
                     <horizontal>
@@ -91,12 +97,5 @@
                     <resolution>0.01</resolution>
                 </range>
-            </ray>
-            <plugin name="laser_controller" filename="libgazebo_ros_ray_sensor.so">
-                <ros>
-                    <remapping>~/out:=scan</remapping>
-                </ros>
-                <output_type>sensor_msgs/LaserScan</output_type>
-                <frame_name>lidar_link</frame_name>
-            </plugin>
+            </lidar>
         </sensor>
     </gazebo>

File: mirte_description/mirte_master_description/urdf/mirte_master_base.gazebo.xacro (robot description, xacro)
@@ -2,4 +2,8 @@
 <robot xmlns:xacro="http://ros.org/wiki/xacro">
  <xacro:if value="$(arg imu_enable)">
+  <plugin
+    filename="gz-sim-imu-system"
+    name="gz::sim::systems::Imu">
+  </plugin>
   <gazebo reference="imu_link">
     <gravity>true</gravity>
@@ -9,14 +13,4 @@
       <visualize>true</visualize>
       <topic>__default_topic__</topic>
-      <plugin filename="libgazebo_ros_imu_sensor.so" name="imu_plugin">
-        <topicName>imu</topicName>
-        <bodyName>imu_link</bodyName>
-        <updateRateHZ>10.0</updateRateHZ>
-        <gaussianNoise>0.0</gaussianNoise>
-        <xyzOffset>0 0 0</xyzOffset>
-        <rpyOffset>0 0 0</rpyOffset>
-        <frameName>imu_link</frameName>
-        <initialOrientationAsReference>false</initialOrientationAsReference>
-      </plugin>
       <pose>0 0 0 0 0 0</pose>
     </sensor>

File: mirte_description/mirte_master_description/urdf/orbbec_astra_plus_pro.xacro (robot description, xacro)
@@ -100,8 +100,15 @@
      ========================================================= -->
      <xacro:macro name="sensor_orbbec_astra_pro_plus_gazebo">
+          <plugin
+               filename="gz-sim-sensors-system"
+               name="gz::sim::systems::Sensors">
+               <render_engine>ogre2</render_engine>
+          </plugin>
           <gazebo reference="${name}_link">
-             <sensor name="${name}" type="depth">
+             <sensor name="${name}" type="rgbd_camera">
                 <visualize>true</visualize>
                 <update_rate>60.0</update_rate>
+                <alwaysOn>true</alwaysOn>
+                <topic>rgbd_camera</topic>
                 <camera name="RS_D455">
                     <horizontal_fov>${60.0*M_PI/180.0}</horizontal_fov>
@@ -115,23 +122,13 @@
                         <far>10.0</far>
                     </clip>
+                    <distorsion>
+                         <k1>0.0</k1>
+                         <k2>0.0</k2>
+                         <k3>0.0</k3>
+                         <p1>0.0</p1>
+                         <p2>0.0</p2>
+                    </distorsion>
+                    <optical_frame_id>camera_link</optical_frame_id>
                 </camera>
-                <plugin name="${name}_controller" filename="libgazebo_ros_camera.so">
-                    <baseline>0.1</baseline>
-                    <alwaysOn>true</alwaysOn>
-                    <updateRate>30</updateRate>
-                    <frame_name>${name}_depth_optical_frame</frame_name>
-                    <pointCloudCutoff>0.6</pointCloudCutoff>
-                    <pointCloudCutoffMax>8.0</pointCloudCutoffMax>
-                    <distortionK1>0</distortionK1>
-                    <distortionK2>0</distortionK2>
-                    <distortionK3>0</distortionK3>
-                    <distortionT1>0</distortionT1>
-                    <distortionT2>0</distortionT2>
-                    <CxPrime>0</CxPrime>
-                    <Cx>0</Cx>
-                    <Cy>0</Cy>
-                    <focalLength>0</focalLength>
-                    <hackBaseline>0</hackBaseline>
-                </plugin>
             </sensor>
          </gazebo>

File: mirte_description/mirte_master_description/urdf/ros2_control.xacro (robot description, xacro)
@@ -14,5 +14,5 @@
       <hardware>
         <xacro:if value="$(arg sim)">
-          <plugin>gazebo_ros2_control/GazeboSystem</plugin>
+          <plugin>gz_ros2_control/GazeboSimSystem</plugin>
         </xacro:if>
         <xacro:unless value="$(arg sim)">
@@ -35,5 +35,5 @@
       <hardware>
         <xacro:if value="$(arg sim)">
-          <plugin>gazebo_ros2_control/GazeboSystem</plugin>
+          <plugin>gz_ros2_control/GazeboSimSystem</plugin>
         </xacro:if>
         <xacro:unless value="$(arg sim)">
@@ -71,5 +71,5 @@
      <hardware>
         <xacro:if value="$(arg sim)">
-          <plugin>gazebo_ros2_control/GazeboSystem</plugin>
+          <plugin>gz_ros2_control/GazeboSimSystem</plugin>
         </xacro:if>
         <xacro:unless value="$(arg sim)">
@@ -84,5 +84,4 @@
     <xacro:if value="$(arg sim)">
       <joint name="_Gripper_joint_r">
-        <param name="mimic">gripper_joint</param>
         <param name="multiplier">-1</param>
         <command_interface name="position"/>
@@ -91,5 +90,4 @@
       </joint>
       <joint name="_gripper_link_joint_l">
-        <param name="mimic">gripper_joint</param>
         <param name="multiplier">-1.4</param>
         <command_interface name="position"/>
@@ -98,5 +96,4 @@
       </joint>
       <joint name="_gripper_link_joint_r">
-        <param name="mimic">gripper_joint</param>
         <param name="multiplier">1.4</param>
         <command_interface name="position"/>
@@ -107,5 +104,5 @@
 </ros2_control>
 <gazebo>
-    <plugin filename="libgazebo_ros2_control.so" name="gazebo_ros2_control">
+    <plugin filename="libgz_ros2_control-system.so" name="gz_ros2_control::GazeboSimROS2ControlPlugin">
        <parameters>$(find mirte_base_control)/config/mirte_base_control.yaml</parameters>
        <xacro:if value="$(arg arm_enable)">
@@ -113,17 +110,23 @@
        </xacro:if>
     </plugin>
-    <plugin filename="libgazebo_ros_planar_move.so" name="gazebo_planar_move">
-       <robot_base_frame>base_link</robot_base_frame>
+    <plugin
+      filename="gz-sim-mecanum-drive-system"
+      name="gz::sim::systems::MecanumDrive">
+      <front_left_joint>front_left_wheel_joint</front_left_joint>
+      <front_right_joint>front_right_wheel_joint</front_right_joint>
+      <back_left_joint>rear_left_wheel_joint</back_left_joint>
+      <back_right_joint>rear_right_wheel_joint</back_right_joint>
+      <wheel_separation>1.25</wheel_separation>
+      <wheelbase>1.511</wheelbase>
+      <wheel_radius>0.3</wheel_radius>
+      <min_acceleration>-5</min_acceleration>
+      <max_acceleration>5</max_acceleration>
+      <topic>cmd_vel</topic>
+      <odom_topic>odom</odom_topic>
+      <frame_id>odom</frame_id>
+      <child_frame_id>base_footprint</child_frame_id>
+      <odom_publisher_frequency>30</odom_publisher_frequency>
+      <tf_topic>/tf</tf_topic>
     </plugin>
-    <plugin name="libgazebo_ros_p3d" filename="libgazebo_ros_p3d.so">
-        <ros>
-            <namespace>groundtruth</namespace>
-            <remapping>odom:=odom</remapping>
-        </ros>
-        <frame_name>world</frame_name>
-        <body_name>base_link</body_name>
-        <update_rate>200.0</update_rate>
-        <gaussian_noise>0.0</gaussian_noise>
-     </plugin>
 </gazebo>
 </robot>

File: mirte_description/mirte_master_description/urdf/ultrasonic.xacro (robot description, xacro)
@@ -26,8 +26,15 @@
       </collision>
     </link>
+    <plugin
+      filename="gz-sim-sensors-system"
+      name="gz::sim::systems::Sensors">
+      <render_engine>ogre2</render_engine>
+    </plugin>
     <gazebo reference="${name}_sonar">
-      <sensor type="ray" name="range_sensor_${name}">
+      <sensor type="gpu_lidar" name="range_sensor_${name}">
         <visualize>${visualize_sensors}</visualize>
-          <ray>
+        <always_on>true</always_on>
+        <topic>distance/${name}</topic>
+          <lidar>
             <scan>
               <horizontal>
@@ -56,15 +63,7 @@
            <stddev>0.01</stddev>
          </noise>
-       </ray>
+       </lidar>
        <!-- Using gazebo's update rate instead of plugin's -->
        <update_rate>30</update_rate>
-       <plugin name="gazebo_ros_range_controller_${name}" filename="libgazebo_ros_ray_sensor.so">
-         <ros>
-           <namespace>/mirte</namespace>
-           <remapping>~/out:=distance/${name}</remapping>
-         </ros>
-         <output_type>sensor_msgs/Range</output_type>
-         <radiation_type>ultrasound</radiation_type>
-       </plugin>
      </sensor>
    </gazebo>

Commit message: Revert "Support with gz harmonic"

File: mirte_description/mirte_master_description/urdf/arm.xacro (robot description, xacro)
@@ -353,4 +353,5 @@
             effort="0.0"
             velocity="0.0" />
+        <mimic joint="gripper_joint" multiplier="1.4"/>
     </joint>
     <link
@@ -464,4 +465,5 @@
             effort="0.0"
             velocity="0.0" />
+        <mimic joint="gripper_joint" multiplier="-1.4"/>
     </joint>
     <link
@@ -576,4 +578,5 @@
             velocity="2.0"
         />
+        <mimic joint="gripper_joint" multiplier="-1"/>
     </joint>
 <gazebo>

File: mirte_description/mirte_master_description/urdf/lidar.xacro (robot description, xacro)
@@ -72,17 +72,10 @@
     <xacro:property name="lidar_sensor_link" value="lidar_link" />
   </xacro:unless>
-  <plugin
-    filename="gz-sim-sensors-system"
-    name="gz::sim::systems::Sensors">
-    <render_engine>ogre2</render_engine>
-  </plugin>
   <gazebo reference="lidar_link">
-        <sensor name="lidar" type="gpu_lidar">
-            <always_on>true</always_on>
-            <gz_frame_id>lidar_link</gz_frame_id>
+        <sensor name="lidar" type="ray">
+            <pose> 0 0 0 0 0 0 </pose>
             <visualize>${visualize_sensors}</visualize>
             <update_rate>10</update_rate>
-            <topic>scan</topic>
-            <lidar>
+            <ray>
                 <scan>
                     <horizontal>
@@ -98,5 +91,12 @@
                     <resolution>0.01</resolution>
                 </range>
-            </lidar>
+            </ray>
+            <plugin name="laser_controller" filename="libgazebo_ros_ray_sensor.so">
+                <ros>
+                    <remapping>~/out:=scan</remapping>
+                </ros>
+                <output_type>sensor_msgs/LaserScan</output_type>
+                <frame_name>lidar_link</frame_name>
+            </plugin>
         </sensor>
     </gazebo>

File: mirte_description/mirte_master_description/urdf/mirte_master_base.gazebo.xacro (robot description, xacro)
@@ -2,8 +2,4 @@
 <robot xmlns:xacro="http://ros.org/wiki/xacro">
  <xacro:if value="$(arg imu_enable)">
-  <plugin
-    filename="gz-sim-imu-system"
-    name="gz::sim::systems::Imu">
-  </plugin>
   <gazebo reference="imu_link">
     <gravity>true</gravity>
@@ -13,4 +9,14 @@
       <visualize>true</visualize>
       <topic>__default_topic__</topic>
+      <plugin filename="libgazebo_ros_imu_sensor.so" name="imu_plugin">
+        <topicName>imu</topicName>
+        <bodyName>imu_link</bodyName>
+        <updateRateHZ>10.0</updateRateHZ>
+        <gaussianNoise>0.0</gaussianNoise>
+        <xyzOffset>0 0 0</xyzOffset>
+        <rpyOffset>0 0 0</rpyOffset>
+        <frameName>imu_link</frameName>
+        <initialOrientationAsReference>false</initialOrientationAsReference>
+      </plugin>
       <pose>0 0 0 0 0 0</pose>
     </sensor>

File: mirte_description/mirte_master_description/urdf/orbbec_astra_plus_pro.xacro (robot description, xacro)
@@ -100,15 +100,8 @@
      ========================================================= -->
      <xacro:macro name="sensor_orbbec_astra_pro_plus_gazebo">
-          <plugin
-               filename="gz-sim-sensors-system"
-               name="gz::sim::systems::Sensors">
-               <render_engine>ogre2</render_engine>
-          </plugin>
           <gazebo reference="${name}_link">
-             <sensor name="${name}" type="rgbd_camera">
+             <sensor name="${name}" type="depth">
                 <visualize>true</visualize>
                 <update_rate>60.0</update_rate>
-                <alwaysOn>true</alwaysOn>
-                <topic>rgbd_camera</topic>
                 <camera name="RS_D455">
                     <horizontal_fov>${60.0*M_PI/180.0}</horizontal_fov>
@@ -122,13 +115,23 @@
                         <far>10.0</far>
                     </clip>
-                    <distorsion>
-                         <k1>0.0</k1>
-                         <k2>0.0</k2>
-                         <k3>0.0</k3>
-                         <p1>0.0</p1>
-                         <p2>0.0</p2>
-                    </distorsion>
-                    <optical_frame_id>camera_link</optical_frame_id>
                 </camera>
+                <plugin name="${name}_controller" filename="libgazebo_ros_camera.so">
+                    <baseline>0.1</baseline>
+                    <alwaysOn>true</alwaysOn>
+                    <updateRate>30</updateRate>
+                    <frame_name>${name}_depth_optical_frame</frame_name>
+                    <pointCloudCutoff>0.6</pointCloudCutoff>
+                    <pointCloudCutoffMax>8.0</pointCloudCutoffMax>
+                    <distortionK1>0</distortionK1>
+                    <distortionK2>0</distortionK2>
+                    <distortionK3>0</distortionK3>
+                    <distortionT1>0</distortionT1>
+                    <distortionT2>0</distortionT2>
+                    <CxPrime>0</CxPrime>
+                    <Cx>0</Cx>
+                    <Cy>0</Cy>
+                    <focalLength>0</focalLength>
+                    <hackBaseline>0</hackBaseline>
+                </plugin>
             </sensor>
          </gazebo>

File: mirte_description/mirte_master_description/urdf/ros2_control.xacro (robot description, xacro)
@@ -14,5 +14,5 @@
       <hardware>
         <xacro:if value="$(arg sim)">
-          <plugin>gz_ros2_control/GazeboSimSystem</plugin>
+          <plugin>gazebo_ros2_control/GazeboSystem</plugin>
         </xacro:if>
         <xacro:unless value="$(arg sim)">
@@ -35,5 +35,5 @@
       <hardware>
         <xacro:if value="$(arg sim)">
-          <plugin>gz_ros2_control/GazeboSimSystem</plugin>
+          <plugin>gazebo_ros2_control/GazeboSystem</plugin>
         </xacro:if>
         <xacro:unless value="$(arg sim)">
@@ -71,5 +71,5 @@
      <hardware>
         <xacro:if value="$(arg sim)">
-          <plugin>gz_ros2_control/GazeboSimSystem</plugin>
+          <plugin>gazebo_ros2_control/GazeboSystem</plugin>
         </xacro:if>
         <xacro:unless value="$(arg sim)">
@@ -84,4 +84,5 @@
     <xacro:if value="$(arg sim)">
       <joint name="_Gripper_joint_r">
+        <param name="mimic">gripper_joint</param>
         <param name="multiplier">-1</param>
         <command_interface name="position"/>
@@ -90,4 +91,5 @@
       </joint>
       <joint name="_gripper_link_joint_l">
+        <param name="mimic">gripper_joint</param>
         <param name="multiplier">-1.4</param>
         <command_interface name="position"/>
@@ -96,4 +98,5 @@
       </joint>
       <joint name="_gripper_link_joint_r">
+        <param name="mimic">gripper_joint</param>
         <param name="multiplier">1.4</param>
         <command_interface name="position"/>
@@ -104,5 +107,5 @@
 </ros2_control>
 <gazebo>
-    <plugin filename="libgz_ros2_control-system.so" name="gz_ros2_control::GazeboSimROS2ControlPlugin">
+    <plugin filename="libgazebo_ros2_control.so" name="gazebo_ros2_control">
        <parameters>$(find mirte_base_control)/config/mirte_base_control.yaml</parameters>
        <xacro:if value="$(arg arm_enable)">
@@ -110,23 +113,17 @@
        </xacro:if>
     </plugin>
-    <plugin
-      filename="gz-sim-mecanum-drive-system"
-      name="gz::sim::systems::MecanumDrive">
-      <front_left_joint>front_left_wheel_joint</front_left_joint>
-      <front_right_joint>front_right_wheel_joint</front_right_joint>
-      <back_left_joint>rear_left_wheel_joint</back_left_joint>
-      <back_right_joint>rear_right_wheel_joint</back_right_joint>
-      <wheel_separation>1.25</wheel_separation>
-      <wheelbase>1.511</wheelbase>
-      <wheel_radius>0.3</wheel_radius>
-      <min_acceleration>-5</min_acceleration>
-      <max_acceleration>5</max_acceleration>
-      <topic>cmd_vel</topic>
-      <odom_topic>odom</odom_topic>
-      <frame_id>odom</frame_id>
-      <child_frame_id>base_footprint</child_frame_id>
-      <odom_publisher_frequency>30</odom_publisher_frequency>
-      <tf_topic>/tf</tf_topic>
+    <plugin filename="libgazebo_ros_planar_move.so" name="gazebo_planar_move">
+       <robot_base_frame>base_link</robot_base_frame>
     </plugin>
+    <plugin name="libgazebo_ros_p3d" filename="libgazebo_ros_p3d.so">
+        <ros>
+            <namespace>groundtruth</namespace>
+            <remapping>odom:=odom</remapping>
+        </ros>
+        <frame_name>world</frame_name>
+        <body_name>base_link</body_name>
+        <update_rate>200.0</update_rate>
+        <gaussian_noise>0.0</gaussian_noise>
+     </plugin>
 </gazebo>
 </robot>

File: mirte_description/mirte_master_description/urdf/ultrasonic.xacro (robot description, xacro)
@@ -26,15 +26,8 @@
       </collision>
     </link>
-    <plugin
-      filename="gz-sim-sensors-system"
-      name="gz::sim::systems::Sensors">
-      <render_engine>ogre2</render_engine>
-    </plugin>
     <gazebo reference="${name}_sonar">
-      <sensor type="gpu_lidar" name="range_sensor_${name}">
+      <sensor type="ray" name="range_sensor_${name}">
         <visualize>${visualize_sensors}</visualize>
-        <always_on>true</always_on>
-        <topic>distance/${name}</topic>
-          <lidar>
+          <ray>
             <scan>
               <horizontal>
@@ -63,7 +56,15 @@
            <stddev>0.01</stddev>
          </noise>
-       </lidar>
+       </ray>
        <!-- Using gazebo's update rate instead of plugin's -->
        <update_rate>30</update_rate>
+       <plugin name="gazebo_ros_range_controller_${name}" filename="libgazebo_ros_ray_sensor.so">
+         <ros>
+           <namespace>/mirte</namespace>
+           <remapping>~/out:=distance/${name}</remapping>
+         </ros>
+         <output_type>sensor_msgs/Range</output_type>
+         <radiation_type>ultrasound</radiation_type>
+       </plugin>
      </sensor>
    </gazebo>

Commit message: Add gripper camera for mmv3 urdf, thanks @JakaHatlakLJ

File: mirte_description/mirte_master_description/urdf/arm.xacro (robot description, xacro)
@@ -579,4 +579,12 @@
         />
         <mimic joint="gripper_joint" multiplier="-1"/>
+    </joint>
+    <link name="gripper_camera_link" />
+    <joint name="gripper_camera_joint" type="fixed">
+        <origin
+            xyz="0.027 0 -0.067"
+            rpy="1.5707963267949 0 1.5707963267949" />
+        <parent link="wrist" />
+        <child link="gripper_camera_link" />
     </joint>
 <gazebo>
