Commit message: Working version for arm and base, still TF issues

File: mirte_control/mirte_master_base_control/bringup/urdf/base.urdf.xacro (robot description, xacro)
@@ -31,5 +31,5 @@
         <xacro:wheel name="right_rear" prefix="$(arg prefix)" />
         <xacro:wheel name="right_front" prefix="$(arg prefix)" />
-            <ros2_control name="mecanumdrive" type="system">
+   <ros2_control name="mecanumdrive" type="system">
       <hardware>
         <plugin>mirte_base_control/MirteBaseHWInterface</plugin>
@@ -46,17 +46,4 @@
         <xacro:joint prefix="$(arg prefix)" name="left_rear"  />
         <xacro:joint prefix="$(arg prefix)" name="right_rear"  />
-      <!-- <joint name="${prefix}right_wheel_joint">
-        <command_interface name="velocity"/>
-        <state_interface name="position"/>
-        <state_interface name="velocity"/>
-      </joint> -->
     </ros2_control>
-  <!-- <xacro:include filename="$(find mirte_control)/urdf/diffbot_description.urdf.xacro" />
-  <!- -  Import Rviz colors - ->
-  <xacro:include filename="$(find mirte_control)/urdf/diffbot.materials.xacro" />
-  <!- - Import diffbot ros2_control description - ->
-  <xacro:include filename="$(find mirte_control)/ros2_control/diffbot.ros2_control.xacro" />
-  <xacro:diffbot prefix="$(arg prefix)" />
-  <xacro:diffbot_ros2_control
-    name="DiffBot" prefix="$(arg prefix)" /> -->
 </robot>

File: mirte_description/mirte_master_description/urdf/arm.xacro (robot description, xacro)
@@ -2,5 +2,5 @@
 <robot xmlns:xacro="http://www.ros.org/wiki/xacro">
     <link
-        name="arm_shoulder_pan">
+        name="shoulder_pan">
         <inertial>
             <origin
@@ -42,5 +42,5 @@
     </link>
     <joint
-        name="arm_shoulder_pan_joint"
+        name="shoulder_pan_joint"
         type="revolute">
         <origin
@@ -50,5 +50,5 @@
             link="frame_link" />
         <child
-            link="arm_shoulder_pan" />
+            link="shoulder_pan" />
         <axis
             xyz="0 1 0" />
@@ -61,5 +61,5 @@
     </joint>
     <link
-        name="arm_shoulder_lift">
+        name="shoulder_lift">
         <inertial>
             <origin
@@ -101,5 +101,5 @@
     </link>
     <joint
-        name="arm_shoulder_lift_joint"
+        name="shoulder_lift_joint"
         type="revolute">
         <origin
@@ -107,7 +107,7 @@
             rpy="3.1416 0 1.5708" />
         <parent
-            link="arm_shoulder_pan" />
-        <child
-            link="arm_shoulder_lift" />
+            link="shoulder_pan" />
+        <child
+            link="shoulder_lift" />
         <axis
             xyz="0 1 0" />
@@ -120,5 +120,5 @@
     </joint>
     <link
-        name="arm_elbow">
+        name="elbow">
         <inertial>
             <origin
@@ -160,5 +160,5 @@
     </link>
     <joint
-        name="arm_elbow_joint"
+        name="elbow_joint"
         type="revolute">
         <origin
@@ -166,7 +166,7 @@
             rpy="-3.1416 0 1.5708" />
         <parent
-            link="arm_shoulder_lift" />
-        <child
-            link="arm_elbow" />
+            link="shoulder_lift" />
+        <child
+            link="elbow" />
         <axis
             xyz="1 0 0" />
@@ -179,5 +179,5 @@
     </joint>
     <link
-        name="arm_wrist">
+        name="wrist">
         <inertial>
             <origin
@@ -219,5 +219,5 @@
     </link>
     <joint
-        name="arm_wrist_joint"
+        name="wrist_joint"
         type="revolute">
         <origin
@@ -225,7 +225,7 @@
             rpy="3.1416 0 1.5708" />
         <parent
-            link="arm_elbow" />
-        <child
-            link="arm_wrist" />
+            link="elbow" />
+        <child
+            link="wrist" />
         <axis
             xyz="0 1 0" />
@@ -284,5 +284,5 @@
             rpy="-1.5708 0 0" />
         <parent
-            link="arm_wrist" />
+            link="wrist" />
         <child
             link="gripper" />
@@ -343,5 +343,5 @@
             rpy="1.5708 0 -1.3641" />
         <parent
-            link="arm_wrist" />
+            link="wrist" />
         <child
             link="_gripper_link_r" />
@@ -353,5 +353,5 @@
             effort="0.0"
             velocity="0.0" />
-        <mimic joint="Gripper_joint" multiplier="1.4"/>
+        <mimic joint="gripper_joint" multiplier="1.4"/>
     </joint>
     <link
@@ -460,5 +460,5 @@
             rpy="1.5708 0 -1.7775" />
         <parent
-            link="arm_wrist" />
+            link="wrist" />
         <child
             link="_gripper_link_l" />
@@ -470,5 +470,5 @@
             effort="0.0"
             velocity="0.0" />
-        <mimic joint="Gripper_joint" multiplier="-1.4"/>
+        <mimic joint="gripper_joint" multiplier="-1.4"/>
     </joint>
     <link
@@ -577,5 +577,5 @@
             rpy="-1.5708 0 -3.1416" />
         <parent
-            link="arm_wrist" />
+            link="wrist" />
         <child
             link="_Gripper_r" />
@@ -594,5 +594,5 @@
        <arm>
           <arm_name>finger_gripper</arm_name>
-          <palm_link>arm_wrist</palm_link>
+          <palm_link>wrist</palm_link>
           <gripper_link>gripper</gripper_link>
           <gripper_link>_Gripper_r</gripper_link>

File: mirte_description/mirte_master_description/urdf/ros2_control.xacro (robot description, xacro)
@@ -1,5 +1,42 @@
 <?xml version="1.0"?>
 <robot xmlns:xacro="http://www.ros.org/wiki/xacro">
-<!--
+   <xacro:property name="yaml_param_file" value="$(find mirte_base_control)/config/control_master.yaml"/>
+    <xacro:property name="params" value="${xacro.load_yaml(yaml_param_file)}"/>
+<xacro:arg name="prefix" default="" />
+<xacro:macro name="wheel" params="name prefix">
+        <joint name="${prefix}${name}_wheel_joint" type="continuous">
+      <parent link="${prefix}base_link"/>
+      <child link="${prefix}${name}_wheel"/>
+      <origin xyz="0 0 0" rpy="0 0 0"/>
+      <axis xyz="0 1 0"/>
+      <dynamics damping="0.2"/>
+    </joint>
+    <!-- left wheel Link -->
+    <link name="${prefix}${name}_wheel">
+</link>
+</xacro:macro>
+<xacro:macro name="joint" params="name prefix">
+      <joint name="${prefix}${name}_wheel_joint">
+        <command_interface name="velocity"/>
+        <state_interface name="position"/>
+        <state_interface name="velocity"/>
+      </joint>
+</xacro:macro>
+   <ros2_control name="mecanumdrive" type="system">
+      <hardware>
+        <plugin>mirte_base_control/MirteBaseHWInterface</plugin>
+        <param name="ticks">${params['ticks']}</param>
+        <param name="enable_pid">${params['enable_pid']}</param>
+        <param name="kp">${params['kp']}</param>
+        <param name="ki">${params['ki']}</param>
+        <param name="kd">${params['kd']}</param>
+        <param name="i_clamp">${params['i_clamp']}</param>
+        <param name="antiwindup">${params['antiwindup']}</param>
+      </hardware>
+      <xacro:joint prefix="$(arg prefix)" name="left_front"  />
+        <xacro:joint prefix="$(arg prefix)" name="right_front"  />
+        <xacro:joint prefix="$(arg prefix)" name="left_rear"  />
+        <xacro:joint prefix="$(arg prefix)" name="right_rear"  />
+    </ros2_control>
 <ros2_control name="ros2_arm_control" type="system">
       <hardware>
@@ -9,10 +46,10 @@
         <param name="example_param_hw_slowdown">1</param>
       </hardware>
-   <joint name="arm_shoulder_pan_joint">
+   <joint name="shoulder_pan_joint">
         <command_interface name="position"/>
         <state_interface name="position"/>
         <state_interface name="velocity" />
    </joint>
-    <joint name="arm_shoulder_lift_joint">
+    <joint name="shoulder_lift_joint">
         <command_interface name="position"/>
         <state_interface name="position">
@@ -21,5 +58,5 @@
         <state_interface name="velocity" />
     </joint>
-    <joint name="arm_elbow_joint">
+    <joint name="elbow_joint">
         <command_interface name="position"/>
         <state_interface name="position">
@@ -28,5 +65,5 @@
         <state_interface name="velocity" />
     </joint>
-    <joint name="arm_wrist_joint">
+    <joint name="wrist_joint">
         <command_interface name="position"/>
         <state_interface name="position">
@@ -36,5 +73,4 @@
     </joint>
 </ros2_control>
--->
 <ros2_control name="ros2_gripper_control" type="system">
      <hardware>
@@ -125,59 +161,5 @@
         <state_interface name="effort" />
     </joint>
-    <xacro:if value="$(arg arm_enable)">
-    <joint name="arm_Rot_joint">
-        <command_interface name="position"/>
-        <state_interface name="position"/>
-   </joint>
-    <joint name="arm_Shoulder_joint">
-        <command_interface name="position"/>
-        <state_interface name="position">
-          <param name="initial_value">-1.56</param>
-        </state_interface>
-    </joint>
-    <joint name="arm_Elbow_joint">
-        <command_interface name="position"/>
-        <state_interface name="position">
-          <param name="initial_value">-1.56</param>
-        </state_interface>
-    </joint>
-    <joint name="arm_Wrist_joint">
-        <command_interface name="position"/>
-        <state_interface name="position">
-          <param name="initial_value">1.56</param>
-        </state_interface>
-    </joint>
-    <joint name="Gripper_joint">
-        <command_interface name="position"/>
-        <state_interface name="position" />
-    </joint>
-    <joint name="_Gripper_joint_r">
-        <param name="mimic">Gripper_joint</param>
-        <param name="multiplier">-1</param>
-        <command_interface name="position"/>
-        <state_interface name="position" />
-    </joint>
-    <joint name="_gripper_link_joint_l">
-        <param name="mimic">Gripper_joint</param>
-        <param name="multiplier">-1.4</param>
-        <command_interface name="position"/>
-        <state_interface name="position" />
-    </joint>
-    <joint name="_gripper_link_joint_r">
-        <param name="mimic">Gripper_joint</param>
-        <param name="multiplier">1.4</param>
-        <command_interface name="position"/>
-        <state_interface name="position" />
-    </joint>
-    <joint name="gripper_finger_joint_l">
-        <command_interface name="position"/>
-        <state_interface name="position" />
-    </joint>
-    <joint name="gripper_finger_joint_r">
-        <command_interface name="position"/>
-        <state_interface name="position" />
-    </joint>
-    </xacro:if>
-  </ros2_control>
+</ros2_control>
 -->
 <gazebo>

Commit message: Renamed all wheels to <front/rear> <left/right>

File: mirte_control/mirte_master_base_control/bringup/urdf/base.urdf.xacro (robot description, xacro)
@@ -27,8 +27,8 @@
 </link>
 <!-- same ordering as the mecanum drive controller -->
-        <xacro:wheel name="left_front" prefix="$(arg prefix)" />
-        <xacro:wheel name="left_rear" prefix="$(arg prefix)" />
-        <xacro:wheel name="right_rear" prefix="$(arg prefix)" />
-        <xacro:wheel name="right_front" prefix="$(arg prefix)" />
+        <xacro:wheel name="front_left" prefix="$(arg prefix)" />
+        <xacro:wheel name="rear_left" prefix="$(arg prefix)" />
+        <xacro:wheel name="rear_right" prefix="$(arg prefix)" />
+        <xacro:wheel name="front_right" prefix="$(arg prefix)" />
    <ros2_control name="mecanumdrive" type="system">
       <hardware>
@@ -42,8 +42,8 @@
         <param name="antiwindup">${params['antiwindup']}</param>
       </hardware>
-      <xacro:joint prefix="$(arg prefix)" name="left_front"  />
-        <xacro:joint prefix="$(arg prefix)" name="right_front"  />
-        <xacro:joint prefix="$(arg prefix)" name="left_rear"  />
-        <xacro:joint prefix="$(arg prefix)" name="right_rear"  />
+      <xacro:joint prefix="$(arg prefix)" name="front_left"  />
+        <xacro:joint prefix="$(arg prefix)" name="front_right"  />
+        <xacro:joint prefix="$(arg prefix)" name="rear_left"  />
+        <xacro:joint prefix="$(arg prefix)" name="rear_right"  />
     </ros2_control>
 </robot>

File: mirte_description/mirte_master_description/urdf/mirte_master.xacro (robot description, xacro)
@@ -95,5 +95,5 @@
   <xacro:include filename="$(find mirte_master_description)/urdf/wheel.xacro" />
    <!-- 0.025   -1 -->
-    <xacro:mecanum_wheel name="left_front" wheel_type="left" link_origin="0.025">
+    <xacro:mecanum_wheel name="front_left" wheel_type="left" link_origin="0.025">
       <origin
         xyz="${0.153 - 0} -0.085 -0.0455"
@@ -101,5 +101,5 @@
     </xacro:mecanum_wheel>
    <!-- 0.025   -1 -->
-    <xacro:mecanum_wheel name="left_rear" wheel_type="right" link_origin="0.025">
+    <xacro:mecanum_wheel name="rear_left" wheel_type="right" link_origin="0.025">
       <origin
         xyz="${0.153 - 0} 0.085 -0.0455"
@@ -107,5 +107,5 @@
     </xacro:mecanum_wheel>
    <!-- -0.025   -1 -->
-    <xacro:mecanum_wheel name="right_front" wheel_type="right" link_origin="-0.025">
+    <xacro:mecanum_wheel name="front_right" wheel_type="right" link_origin="-0.025">
       <origin
         xyz="${-0.153 + wheel_length} -0.085 -0.0455"
@@ -113,5 +113,5 @@
     </xacro:mecanum_wheel>
    <!-- -0.025   -1 -->
-    <xacro:mecanum_wheel name="right_rear" wheel_type="left" link_origin="-0.025">
+    <xacro:mecanum_wheel name="rear_right" wheel_type="left" link_origin="-0.025">
       <origin
         xyz="${-0.153 + wheel_length} 0.085 -0.0455"

File: mirte_description/mirte_master_description/urdf/mirte_master_base.gazebo.xacro (robot description, xacro)
@@ -28,8 +28,8 @@
   </gazebo>
   <xacro:include filename="$(find mirte_master_description)/urdf/wheel.gazebo.xacro" />
-  <xacro:wheel_gazebo id="left_front" />
-  <xacro:wheel_gazebo id="left_rear" />
-  <xacro:wheel_gazebo id="right_front" />
-  <xacro:wheel_gazebo id="right_rear" />
+  <xacro:wheel_gazebo id="front_left" />
+  <xacro:wheel_gazebo id="rear_left" />
+  <xacro:wheel_gazebo id="front_right" />
+  <xacro:wheel_gazebo id="rear_right" />
   <xacro:include filename="$(find mirte_master_description)/urdf/ros2_control.xacro"/>
 </robot>

File: mirte_description/mirte_master_description/urdf/ros2_control.xacro (robot description, xacro)
@@ -5,5 +5,5 @@
 <xacro:arg name="prefix" default="" />
 <xacro:macro name="wheel" params="name prefix">
-        <joint name="${prefix}${name}_wheel_joint" type="continuous">
+    <joint name="${prefix}${name}_wheel_joint" type="continuous">
       <parent link="${prefix}base_link"/>
       <child link="${prefix}${name}_wheel"/>
@@ -34,8 +34,8 @@
         <param name="antiwindup">${params['antiwindup']}</param>
       </hardware>
-      <xacro:joint prefix="$(arg prefix)" name="left_front"  />
-        <xacro:joint prefix="$(arg prefix)" name="right_front"  />
-        <xacro:joint prefix="$(arg prefix)" name="left_rear"  />
-        <xacro:joint prefix="$(arg prefix)" name="right_rear"  />
+      <xacro:joint prefix="$(arg prefix)" name="front_left"  />
+        <xacro:joint prefix="$(arg prefix)" name="front_right"  />
+        <xacro:joint prefix="$(arg prefix)" name="rear_right"  />
+        <xacro:joint prefix="$(arg prefix)" name="rear_left"  />
     </ros2_control>
 <ros2_control name="ros2_arm_control" type="system">
@@ -120,47 +120,4 @@
 -->
 </ros2_control>
-<!--
-  <ros2_control name="GazeboSystem" type="system">
-    <hardware>
-        <plugin>gazebo_ros2_control/GazeboSystem</plugin>
-    </hardware>
-    <joint name="wheel_left_front_joint">
-        <command_interface name="velocity">
-            <param name="min">-10</param>
-            <param name="max">10</param>
-        </command_interface>
-        <state_interface name="position" />
-        <state_interface name="velocity" />
-        <state_interface name="effort" />
-    </joint>
-    <joint name="wheel_right_front_joint">
-        <command_interface name="velocity">
-            <param name="min">-10</param>
-            <param name="max">10</param>
-        </command_interface>
-        <state_interface name="velocity" />
-        <state_interface name="position" />
-        <state_interface name="effort" />
-    </joint>
-   <joint name="wheel_left_rear_joint">
-        <command_interface name="velocity">
-            <param name="min">-10</param>
-            <param name="max">10</param>
-        </command_interface>
-        <state_interface name="velocity" />
-        <state_interface name="position" />
-        <state_interface name="effort" />
-    </joint>
-   <joint name="wheel_right_rear_joint">
-        <command_interface name="velocity">
-            <param name="min">-10</param>
-            <param name="max">10</param>
-        </command_interface>
-        <state_interface name="velocity" />
-        <state_interface name="position" />
-        <state_interface name="effort" />
-    </joint>
-</ros2_control>
--->
 <gazebo>
     <plugin filename="libgazebo_ros2_control.so" name="gazebo_ros2_control">

File: mirte_description/mirte_master_description/urdf/wheel.xacro (robot description, xacro)
@@ -5,5 +5,5 @@
   <xacro:macro name="mecanum_wheel" params="name *origin link_origin wheel_type">
   <link
-    name="wheel_${name}">
+    name="${name}_wheel">
     <inertial>
       <origin xyz="0 0 ${link_origin}" />
@@ -32,17 +32,17 @@
   </link>
   <joint
-    name="wheel_${name}_joint"
+    name="${name}_wheel_joint"
     type="continuous">
     <xacro:insert_block name="origin"/>
     <parent link="frame_link" />
-    <child link="wheel_${name}" />
+    <child link="${name}_wheel" />
     <axis xyz="0 0 -1" />
   </joint>
-  <transmission name="wheel_${name}_transmission">
+  <transmission name="${name}_wheel_transmission">
     <type>transmission_interface/SimpleTransmission</type>
-    <joint name="wheel_${name}_joint">
+    <joint name="${name}_wheel_joint">
       <hardwareInterface>hardware_interface/VelocityJointInterface</hardwareInterface>
     </joint>
-    <actuator name="wheel_${name}_actuator">
+    <actuator name="${name}_wheel_actuator">
       <mechanicalReduction>1</mechanicalReduction>
     </actuator>

Commit message: Add configurable ticks and invert motors

File: mirte_control/mirte_master_base_control/bringup/urdf/base.urdf.xacro (robot description, xacro)
@@ -4,5 +4,6 @@
     <xacro:property name="yaml_param_file" value="$(find mirte_base_control)/config/control_master.yaml"/>
     <xacro:property name="params" value="${xacro.load_yaml(yaml_param_file)}"/>
-<xacro:macro name="wheel" params="name prefix">
+    <xacro:arg name="ticks" default="${params['ticks']}"/>
+<xa cro:macro name="wheel" params="name prefix">
         <joint name="${prefix}${name}_wheel_joint" type="continuous">
       <parent link="${prefix}base_link"/>
@@ -34,5 +35,5 @@
       <hardware>
         <plugin>mirte_base_control/MirteBaseHWInterface</plugin>
-        <param name="ticks">${params['ticks']}</param>
+        <param name="ticks">$(arg ticks)</param>
         <param name="separate_update_format">${params['separate_update_format']}</param>
         <!-- Use %s in format strings to replace with joint names -->

File: mirte_description/mirte_master_description/urdf/ros2_control.xacro (robot description, xacro)
@@ -4,4 +4,5 @@
 <xacro:property name="params" value="${xacro.load_yaml(yaml_param_file)}"/>
 <xacro:arg name="prefix" default="" />
+<xacro:arg name="ticks" default="${params['ticks']}" />
 <xacro:macro name="joint" params="name prefix">
       <joint name="${prefix}${name}_wheel_joint">
@@ -18,5 +19,5 @@
         <xacro:unless value="$(arg sim)">
           <plugin>mirte_base_control/MirteBaseHWInterface</plugin>
-          <param name="ticks">${params['ticks']}</param>
+          <param name="ticks">$(arg ticks)</param>
         <param name="separate_update_format">${params['separate_update_format']}</param>
         <!-- Use %s in format strings to replace with joint names -->

Commit message: Fix xacro base typo

File: mirte_control/mirte_master_base_control/bringup/urdf/base.urdf.xacro (robot description, xacro)
@@ -5,5 +5,5 @@
     <xacro:property name="params" value="${xacro.load_yaml(yaml_param_file)}"/>
     <xacro:arg name="ticks" default="${params['ticks']}"/>
-<xa cro:macro name="wheel" params="name prefix">
+<xacro:macro name="wheel" params="name prefix">
         <joint name="${prefix}${name}_wheel_joint" type="continuous">
       <parent link="${prefix}base_link"/>
